Commit message: 22 july 2025

File: src/my_rob_con/my_rob_con/task4/urdf/robot2.urdf (robot description, URDF)
Before this commit: robot robot2, 6 links, 5 joints
Links:
- removed link caster_wheel
- removed link front_left_wheel
- removed link front_right_wheel
- removed link rear_left_wheel
- removed link rear_right_wheel
- added link base_footprint
- added link left_back_wheel, mass 0.5; collision cylinder length=0.05 radius=0.1; visual cylinder length=0.05 radius=0.1
- added link left_front_wheel; visual cylinder length=0.05 radius=0.1
- added link lidar; visual cylinder length=0.05 radius=0.05
- added link right_back_wheel, mass 0.5; collision cylinder length=0.05 radius=0.1; visual cylinder length=0.05 radius=0.1
- added link right_front_wheel; visual cylinder length=0.05 radius=0.1
- link base_link: mass 5.0 -> 5; geometry collision box size=0.6 0.4 0.2; visual box size=0.6 0.4 0.2
Joints:
- removed joint caster_joint
- removed joint front_left_wheel_joint
- removed joint front_right_wheel_joint
- removed joint rear_left_wheel_joint
- removed joint rear_right_wheel_joint
- added joint base_joint: type fixed, parent base_footprint, child base_link, origin xyz=0 0 0
- added joint left_back_wheel_joint: type continuous, parent base_link, child left_back_wheel, origin xyz=-0.15 0.225 0, axis 0 1 0
- added joint left_front_wheel_joint: type fixed, parent base_link, child left_front_wheel, origin xyz=0.15 0.225 0
- added joint lidar_joint: type fixed, parent base_link, child lidar, origin xyz=0 0 0.225
- added joint right_back_wheel_joint: type continuous, parent base_link, child right_back_wheel, origin xyz=-0.15 -0.225 0, axis 0 1 0
- added joint right_front_wheel_joint: type fixed, parent base_link, child right_front_wheel, origin xyz=0.15 -0.225 0
